File: DUBEC.sch (EAGLE design)
At the start: 49 parts

Commit message: MCU capacitor
Parts:
- removed CAP_5V: 1.5F, dubec:CAPPOWERSTOR_1.5F
- removed RTOP: 1MOhm, jne:RESR0402
- added 12V_RTOP: 1MOhm, jne:RESR0402
- added 5V_COUT: (no value), dubec:CAP1210
- added MCU_C: (no value), dubec:CAP0508
- 5V_CBIAS: value 4.7uF -> 4.7pF; device jne:CAPC0603 -> dubec:CAP0402
- D12V, D5V_ISP, D_RELAY: value SCH_DIODESCHOTTKY-0402 -> SCH_DIODE; device dubec:SCH_DIODESCHOTTKY-0402 -> dubec:SCH_DIODE
- R_DIV_1, R_DIV_2: device dubec:RESR0402 -> dubec:RES0402
- ZD_DIV: device dubec:Z-DIODE -> dubec:Z-DIODE0503
- renumbered MC to MCU
Connections:
- net 12V: now also 12V_RTOP.1; no longer RTOP.1
- net 5V: now also 5V_COUT.V+; no longer CAP_5V.V+
- net 5V_ISP: now also MCU_C.V+
- net GND: now also 5V_COUT.GND, MCU_C.GND; no longer CAP_5V.GND
- net N$14: now also 12V_RTOP.GND; no longer RTOP.GND
Other:
- note added: "BOM: MCU = ATTINY13A-MMF MCU_C = 298W106X06R3K2T DC_C1, DC_C2, 12V_CO = C2012X5R1V226M125AC 5V_C2 = C1608JB1V475K080AC 5V_CBIAS = GRM1555C1E4R7BA01D 5V_FB1 = 742792012 5V_L2 = IHLP2525CZER6R8M01 5V_C3 = C2012JB1V106K085AC 5V_CIN1, 5V_CIN2 = C1005JB1V105K050BC 5V_L1 = IHLP2525CZER2R2M01 [0420CDMCBDS-2R2MC] 5V_R2 = 2x TNPW0402121RBEED 5V_CSS = CGA2B3X7R1V103K050BB 5V_RT = 5-1879215-9 5V_COUT = GRM3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"
- note removed: "BOM: MC = ATTINY13A-MMFR DC_C1, DC_C2, 12V_CO = C2012X5R1V226M125AC 5V_C2, 5V_CBIAS = C1608JB1V475K080AC 5V_FB1 = 742792012 5V_L2 = IHLP2525CZER6R8M01 5V_C3 = C2012JB1V106K085AC 5V_CIN1, 5V_CIN2 = C1005JB1V105K050BC 5V_L1 = IHLP2525CZER2R2M01 [0420CDMCBDS-2R2MC] 5V_R2 = 2x TNPW0402121RBEED 5V_CSS = CGA2B3X7R1V103K050BB 5V_RT = 5-1879215-9 12V_CBST1, 12V_CBST2, 12V_CIN = UMK105B7104KV-FR 12V_L1 = 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"
- moved on the sheet: 12V-1A4, 12V_C3, 12V_CBST1, 12V_CBST2, 12V_CFB, 12V_CFF, 12V_CIN, 12V_CO, 12V_L1, 12V_RBOT, 12V_RFB, 12V_RFF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
