File: DUBEC.brd (EAGLE design)
At the start: 40 x 21.4 mm, 70 parts

Commit message: Tweaks
Routing:
- net SRC_MAIN: track 17.8 -> 15.2 mm
- net GATE_MAIN: track 18.1 -> 19.5 mm
Changed lines of the file:
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@@
 <grid distance="0.125" unitdist="mm" unit="mm" style="lines" multiple="8" display="yes" altdistance="0.0625" altunitdist="mm" altunit="mm"/>
 <layers>
-<layer number="1" name="Top" color="2" fill="1" visible="yes" active="yes"/>
+<layer number="1" name="Top" color="2" fill="1" visible="no" active="yes"/>
 <layer number="2" name="Route2" color="9" fill="1" visible="no" active="yes"/>
 <layer number="3" name="Route3" color="4" fill="3" visible="no" active="no"/>
 <layer number="14" name="Route14" color="1" fill="6" visible="no" active="no"/>
-<layer number="15" name="Route15" color="14" fill="1" visible="no" active="yes"/>
+<layer number="15" name="Route15" color="14" fill="1" visible="yes" active="yes"/>
 <layer number="16" name="Bottom" color="5" fill="1" visible="no" active="yes"/>
 <layer number="17" name="Pads" color="10" fill="1" visible="yes" active="yes"/>
 <layer number="18" name="Vias" color="2" fill="1" visible="yes" active="yes"/>
 <layer number="19" name="Unrouted" color="6" fill="1" visible="yes" active="yes"/>
-<layer number="20" name="Dimension" color="15" fill="1" visible="yes" active="yes"/>
-<layer number="21" name="tPlace" color="15" fill="1" visible="yes" active="yes"/>
+<layer number="20" name="Dimension" color="15" fill="1" visible="no" active="yes"/>
+<layer number="21" name="tPlace" color="15" fill="1" visible="no" active="yes"/>
 <layer number="22" name="bPlace" color="7" fill="1" visible="no" active="yes"/>
-<layer number="23" name="tOrigins" color="15" fill="1" visible="yes" active="yes"/>
+<layer number="23" name="tOrigins" color="15" fill="1" visible="no" active="yes"/>
 <layer number="24" name="bOrigins" color="15" fill="1" visible="no" active="yes"/>
 <layer number="25" name="tNames" color="7" fill="1" visible="no" active="yes"/>
@@
 <layer number="27" name="tValues" color="7" fill="1" visible="no" active="yes"/>
 <layer number="28" name="bValues" color="7" fill="1" visible="no" active="yes"/>
-<layer number="29" name="tStop" color="4" fill="1" visible="yes" active="yes"/>
+<layer number="29" name="tStop" color="4" fill="1" visible="no" active="yes"/>
 <layer number="30" name="bStop" color="7" fill="6" visible="no" active="yes"/>
 <layer number="31" name="tCream" color="7" fill="4" visible="no" active="yes"/>
 <layer number="32" name="bCream" color="7" fill="5" visible="no" active="yes"/>
-<layer number="33" name="tFinish" color="6" fill="3" visible="yes" active="yes"/>
+<layer number="33" name="tFinish" color="6" fill="3" visible="no" active="yes"/>
 <layer number="34" name="bFinish" color="6" fill="6" visible="no" active="yes"/>
-<layer number="35" name="tGlue" color="7" fill="4" visible="yes" active="yes"/>
+<layer number="35" name="tGlue" color="7" fill="4" visible="no" active="yes"/>
 <layer number="36" name="bGlue" color="7" fill="5" visible="no" active="yes"/>
-<layer number="37" name="tTest" color="7" fill="1" visible="yes" active="yes"/>
+<layer number="37" name="tTest" color="7" fill="1" visible="no" active="yes"/>
 <layer number="38" name="bTest" color="7" fill="1" visible="no" active="yes"/>
-<layer number="39" name="tKeepout" color="4" fill="11" visible="yes" active="yes"/>
+<layer number="39" name="tKeepout" color="4" fill="11" visible="no" active="yes"/>
 <layer number="40" name="bKeepout" color="1" fill="11" visible="no" active="yes"/>
-<layer number="41" name="tRestrict" color="14" fill="10" visible="yes" active="yes"/>
+<layer number="41" name="tRestrict" color="14" fill="10" visible="no" active="yes"/>
 <layer number="42" name="bRestrict" color="1" fill="10" visible="no" active="yes"/>
 <layer number="43" name="vRestrict" color="2" fill="10" visible="no" active="yes"/>
 <layer number="44" name="Drills" color="7" fill="1" visible="no" active="yes"/>
-<layer number="45" name="Holes" color="7" fill="1" visible="yes" active="yes"/>
+<layer number="45" name="Holes" color="7" fill="1" visible="no" active="yes"/>
 <layer number="46" name="Milling" color="3" fill="1" visible="no" active="yes"/>
-<layer number="47" name="Measures" color="7" fill="1" visible="yes" active="yes"/>
+<layer number="47" name="Measures" color="7" fill="1" visible="no" active="yes"/>
 <layer number="48" name="Document" color="7" fill="1" visible="no" active="yes"/>
 <layer number="49" name="Reference" color="7" fill="1" visible="no" active="yes"/>
 <layer number="50" name="dxf" color="7" fill="1" visible="no" active="no"/>
-<layer number="51" name="tDocu" color="7" fill="1" visible="yes" active="yes"/>
+<layer number="51" name="tDocu" color="7" fill="1" visible="no" active="yes"/>
 <layer number="52" name="bDocu" color="7" fill="1" visible="no" active="yes"/>
 <layer number="53" name="tGND_GNDA" color="7" fill="9" visible="no" active="no"/>
@@
 <layer number="100" name="Muster" color="7" fill="1" visible="no" active="no"/>
 <layer number="101" name="Patch_Top" color="12" fill="4" visible="no" active="yes"/>
-<layer number="102" name="tPolarity" color="7" fill="1" visible="yes" active="yes"/>
+<layer number="102" name="tPolarity" color="7" fill="1" visible="no" active="yes"/>
 <layer number="103" name="tMap" color="7" fill="1" visible="no" active="yes"/>
 <layer number="104" name="Name" color="16" fill="1" visible="no" active="yes"/>
-<layer number="105" name="tPlate" color="7" fill="1" visible="yes" active="yes"/>
+<layer number="105" name="tPlate" color="7" fill="1" visible="no" active="yes"/>
 <layer number="106" name="bPlate" color="7" fill="1" visible="no" active="yes"/>
-<layer number="107" name="tLabels" color="15" fill="1" visible="yes" active="yes"/>
+<layer number="107" name="tLabels" color="15" fill="1" visible="no" active="yes"/>
 <layer number="108" name="tplace-old" color="10" fill="1" visible="no" active="yes"/>
 <layer number="109" name="ref-old" color="11" fill="1" visible="no" active="yes"/>
@@
 <polygon width="0.3302" layer="16">
 <vertex x="7.25" y="4.75"/>
-<vertex x="7.25" y="9.125"/>
-<vertex x="11.125" y="13"/>
+<vertex x="7.25" y="9"/>
+<vertex x="11.25" y="13"/>
 <vertex x="17" y="13"/>
 <vertex x="17" y="10.5"/>
@@
 <wire x1="7.975" y1="9.35" x2="7.95" y2="9.375" width="0.3" layer="1"/>
 <wire x1="7.95" y1="9.375" x2="6.625" y2="9.375" width="0.3" layer="1"/>
-<via x="4.75" y="13.125" extent="1-16" drill="0.3"/>
-<wire x1="5.875" y1="9.375" x2="5.625" y2="9.375" width="0.3302" layer="16"/>
-<wire x1="5.625" y1="9.375" x2="4.75" y2="10.25" width="0.3302" layer="16"/>
-<wire x1="4.75" y1="10.25" x2="4.75" y2="13.125" width="0.3302" layer="16"/>
-<wire x1="4.75" y1="13.125" x2="5.5" y2="13.125" width="0.4" layer="1"/>
+<via x="5.5" y="15" extent="1-16" drill="0.3"/>
+<wire x1="5.875" y1="9.375" x2="5.875" y2="14.625" width="0.3302" layer="16"/>
+<wire x1="5.875" y1="14.625" x2="5.5" y2="15" width="0.3302" layer="16"/>
+<wire x1="5.5" y1="15" x2="5.5" y2="14.25" width="0.4" layer="1"/>
 </signal>
 <signal name="GATE_AUX" class="2">
@@
 <via x="14.625" y="16.125" extent="1-16" drill="0.3"/>
 <wire x1="14" y1="16.125" x2="14.625" y2="16.125" width="0.4" layer="1"/>
-<wire x1="2" y1="10.125" x2="3.5" y2="10.125" width="0.3302" layer="15"/>
-<wire x1="3.5" y1="10.125" x2="7.5" y2="14.125" width="0.3302" layer="15"/>
-<wire x1="7.5" y1="14.125" x2="12.625" y2="14.125" width="0.3302" layer="15"/>
-<wire x1="12.625" y1="14.125" x2="14.625" y2="16.125" width="0.3302" layer="15"/>
+<wire x1="2" y1="10.125" x2="4.625" y2="10.125" width="0.3302" layer="15"/>
+<wire x1="4.625" y1="10.125" x2="9.125" y2="14.625" width="0.3302" layer="15"/>
+<wire x1="9.125" y1="14.625" x2="13.125" y2="14.625" width="0.3302" layer="15"/>
+<wire x1="13.125" y1="14.625" x2="14.625" y2="16.125" width="0.3302" layer="15"/>
 </signal>
 <signal name="GATE_MAIN_B" class="2">
@@
 <contactref element="RA1" pad="1"/>
 <contactref element="D2" pad="6"/>
-<via x="5.875" y="10.5" extent="1-16" drill="0.3"/>
-<wire x1="5.875" y1="10.5" x2="6" y2="10.375" width="0.4" layer="1"/>
-<wire x1="6" y1="10.375" x2="6.625" y2="10.375" width="0.4" layer="1"/>
-<wire x1="5.875" y1="10.5" x2="6.25" y2="10.125" width="0.3302" layer="15"/>
-<wire x1="6.25" y1="10.125" x2="8.375" y2="10.125" width="0.3302" layer="15"/>
-<wire x1="8.375" y1="10.125" x2="15" y2="3.5" width="0.3302" layer="15"/>
+<via x="7.5" y="10.5" extent="1-16" drill="0.3"/>
+<wire x1="7.5" y1="10.5" x2="8" y2="10.5" width="0.3302" layer="15"/>
+<wire x1="8" y1="10.5" x2="15" y2="3.5" width="0.3302" layer="15"/>
 <wire x1="15" y1="3.5" x2="15" y2="2.875" width="0.3302" layer="15"/>
-<wire x1="7.975" y1="11.15" x2="7.975" y2="10.725" width="0.3" layer="1"/>
-<wire x1="7.975" y1="10.725" x2="7.625" y2="10.375" width="0.3" layer="1"/>
-<wire x1="7.625" y1="10.375" x2="6.625" y2="10.375" width="0.3" layer="1"/>
+<wire x1="6.625" y1="10.375" x2="7.375" y2="10.375" width="0.4" layer="1"/>
+<wire x1="7.375" y1="10.375" x2="7.5" y2="10.5" width="0.4" layer="1"/>
+<wire x1="7.975" y1="11.15" x2="7.975" y2="10.975" width="0.3" layer="1"/>
+<wire x1="7.975" y1="10.975" x2="7.5" y2="10.5" width="0.3" layer="1"/>
 <wire x1="11.7" y1="4.22" x2="12.8125" y2="3.8125" width="0" layer="19" extent="1-1"/>
 </signal>

Commit message: Tweaks
Parts:
- moved 12TVS 0.25 mm to (31.7, 3.69)
Routing:
- net GND: track 26.2 -> 19.4 mm
- net 12VCC: track 11.9 -> 11.3 mm
- net 12V: track 33.6 -> 33.8 mm, vias 2 -> 3

Commit message: Voltage divider tweak
Parts:
- RAUXBOT: value RES3K_16 -> RES2.94K_16
Changed lines of the file:
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@@
 <grid distance="0.125" unitdist="mm" unit="mm" style="lines" multiple="8" display="yes" altdistance="0.0625" altunitdist="mm" altunit="mm"/>
 <layers>
-<layer number="1" name="Top" color="2" fill="1" visible="no" active="yes"/>
+<layer number="1" name="Top" color="2" fill="1" visible="yes" active="yes"/>
 <layer number="2" name="Route2" color="9" fill="1" visible="no" active="yes"/>
 <layer number="3" name="Route3" color="4" fill="3" visible="no" active="no"/>
 <layer number="14" name="Route14" color="1" fill="6" visible="no" active="no"/>
-<layer number="15" name="Route15" color="14" fill="1" visible="yes" active="yes"/>
+<layer number="15" name="Route15" color="14" fill="1" visible="no" active="yes"/>
 <layer number="16" name="Bottom" color="5" fill="1" visible="no" active="yes"/>
 <layer number="17" name="Pads" color="10" fill="1" visible="yes" active="yes"/>
 <layer number="18" name="Vias" color="2" fill="1" visible="yes" active="yes"/>
 <layer number="19" name="Unrouted" color="6" fill="1" visible="yes" active="yes"/>
-<layer number="20" name="Dimension" color="15" fill="1" visible="no" active="yes"/>
-<layer number="21" name="tPlace" color="15" fill="1" visible="no" active="yes"/>
+<layer number="20" name="Dimension" color="15" fill="1" visible="yes" active="yes"/>
+<layer number="21" name="tPlace" color="15" fill="1" visible="yes" active="yes"/>
 <layer number="22" name="bPlace" color="7" fill="1" visible="no" active="yes"/>
-<layer number="23" name="tOrigins" color="15" fill="1" visible="no" active="yes"/>
+<layer number="23" name="tOrigins" color="15" fill="1" visible="yes" active="yes"/>
 <layer number="24" name="bOrigins" color="15" fill="1" visible="no" active="yes"/>
 <layer number="25" name="tNames" color="7" fill="1" visible="no" active="yes"/>
@@
 <layer number="27" name="tValues" color="7" fill="1" visible="no" active="yes"/>
 <layer number="28" name="bValues" color="7" fill="1" visible="no" active="yes"/>
-<layer number="29" name="tStop" color="4" fill="1" visible="no" active="yes"/>
+<layer number="29" name="tStop" color="4" fill="1" visible="yes" active="yes"/>
 <layer number="30" name="bStop" color="7" fill="6" visible="no" active="yes"/>
 <layer number="31" name="tCream" color="7" fill="4" visible="no" active="yes"/>
 <layer number="32" name="bCream" color="7" fill="5" visible="no" active="yes"/>
-<layer number="33" name="tFinish" color="6" fill="3" visible="no" active="yes"/>
+<layer number="33" name="tFinish" color="6" fill="3" visible="yes" active="yes"/>
 <layer number="34" name="bFinish" color="6" fill="6" visible="no" active="yes"/>
-<layer number="35" name="tGlue" color="7" fill="4" visible="no" active="yes"/>
+<layer number="35" name="tGlue" color="7" fill="4" visible="yes" active="yes"/>
 <layer number="36" name="bGlue" color="7" fill="5" visible="no" active="yes"/>
-<layer number="37" name="tTest" color="7" fill="1" visible="no" active="yes"/>
+<layer number="37" name="tTest" color="7" fill="1" visible="yes" active="yes"/>
 <layer number="38" name="bTest" color="7" fill="1" visible="no" active="yes"/>
-<layer number="39" name="tKeepout" color="4" fill="11" visible="no" active="yes"/>
+<layer number="39" name="tKeepout" color="4" fill="11" visible="yes" active="yes"/>
 <layer number="40" name="bKeepout" color="1" fill="11" visible="no" active="yes"/>
-<layer number="41" name="tRestrict" color="14" fill="10" visible="no" active="yes"/>
+<layer number="41" name="tRestrict" color="14" fill="10" visible="yes" active="yes"/>
 <layer number="42" name="bRestrict" color="1" fill="10" visible="no" active="yes"/>
 <layer number="43" name="vRestrict" color="2" fill="10" visible="no" active="yes"/>
 <layer number="44" name="Drills" color="7" fill="1" visible="no" active="yes"/>
-<layer number="45" name="Holes" color="7" fill="1" visible="no" active="yes"/>
+<layer number="45" name="Holes" color="7" fill="1" visible="yes" active="yes"/>
 <layer number="46" name="Milling" color="3" fill="1" visible="no" active="yes"/>
-<layer number="47" name="Measures" color="7" fill="1" visible="no" active="yes"/>
+<layer number="47" name="Measures" color="7" fill="1" visible="yes" active="yes"/>
 <layer number="48" name="Document" color="7" fill="1" visible="no" active="yes"/>
 <layer number="49" name="Reference" color="7" fill="1" visible="no" active="yes"/>
 <layer number="50" name="dxf" color="7" fill="1" visible="no" active="no"/>
-<layer number="51" name="tDocu" color="7" fill="1" visible="no" active="yes"/>
+<layer number="51" name="tDocu" color="7" fill="1" visible="yes" active="yes"/>
 <layer number="52" name="bDocu" color="7" fill="1" visible="no" active="yes"/>
 <layer number="53" name="tGND_GNDA" color="7" fill="9" visible="no" active="no"/>
@@
 <layer number="100" name="Muster" color="7" fill="1" visible="no" active="no"/>
 <layer number="101" name="Patch_Top" color="12" fill="4" visible="no" active="yes"/>
-<layer number="102" name="tPolarity" color="7" fill="1" visible="no" active="yes"/>
+<layer number="102" name="tPolarity" color="7" fill="1" visible="yes" active="yes"/>
 <layer number="103" name="tMap" color="7" fill="1" visible="no" active="yes"/>
 <layer number="104" name="Name" color="16" fill="1" visible="no" active="yes"/>
-<layer number="105" name="tPlate" color="7" fill="1" visible="no" active="yes"/>
+<layer number="105" name="tPlate" color="7" fill="1" visible="yes" active="yes"/>
 <layer number="106" name="bPlate" color="7" fill="1" visible="no" active="yes"/>
-<layer number="107" name="tLabels" color="15" fill="1" visible="no" active="yes"/>
+<layer number="107" name="tLabels" color="15" fill="1" visible="yes" active="yes"/>
 <layer number="108" name="tplace-old" color="10" fill="1" visible="no" active="yes"/>
 <layer number="109" name="ref-old" color="11" fill="1" visible="no" active="yes"/>
@@
 <attribute name="DIGIKEY_PART_#" value="541-90.9KLCT-ND" x="13.5" y="16.125" size="1.778" layer="27" rot="R180" display="off"/>
 </element>
-<element name="RAUXBOT" library="dubec" package="0402" value="RES3K_16" x="13.5" y="15" rot="R180">
-<attribute name="DIGIKEY_PART_#" value="541-3.00KLCT-ND" x="13.5" y="15" size="1.778" layer="27" rot="R180" display="off"/>
+<element name="RAUXBOT" library="dubec" package="0402" value="RES2.94K_16" x="13.5" y="15" rot="R180">
+<attribute name="DIGIKEY_PART_#" value="541-2.94KLCT-ND" x="13.5" y="15" size="1.778" layer="27" rot="R180" display="off"/>
 <attribute name="MANUFACTURER" value="Vishay Dale" x="13.5" y="15" size="1.778" layer="27" rot="R180" display="off"/>
-<attribute name="MFG_PART_#" value="CRCW04023K00FKED" x="13.5" y="15" size="1.778" layer="27" rot="R180" display="off"/>
+<attribute name="MFG_PART_#" value="CRCW04022K94FKED" x="13.5" y="15" size="1.778" layer="27" rot="R180" display="off"/>
 <attribute name="TOLERANCE" value="±1%" x="13.5" y="15" size="1.778" layer="27" rot="R180" display="off"/>
 <attribute name="TEMP" value="±100ppm/°C" x="13.5" y="15" size="1.778" layer="27" rot="R180" display="off"/>
-<attribute name="EURO" value="2.10/50" x="13.5" y="15" size="1.778" layer="27" rot="R180" display="off"/>
+<attribute name="EURO" value="2.01/50" x="13.5" y="15" size="1.778" layer="27" rot="R180" display="off"/>
 </element>
 <element name="CMCU" library="dubec" package="0402" value="" x="8.25" y="16.875" rot="R90">

Commit message: Voltage divider to 4.6V
Parts:
- RAUXBOT: value RES2.94K_16 -> RES162K_16
- RAUXTOP: value RES90.9K_16 -> RES1M_16
Changed lines of the file:
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@@
 <attribute name="EURO" value="4.06/10" x="31.6875" y="3.6875" size="1.778" layer="27" rot="R270" display="off"/>
 </element>
-<element name="RAUXTOP" library="dubec" package="0402" value="RES90.9K_16" x="13.5" y="16.125" rot="R180">
+<element name="RAUXTOP" library="dubec" package="0402" value="RES1M_16" x="13.5" y="16.125" rot="R180">
 <attribute name="MANUFACTURER" value="Vishay Dale" x="13.5" y="16.125" size="1.778" layer="27" rot="R180" display="off"/>
-<attribute name="MFG_PART_#" value="CRCW040290K9FKED" x="13.5" y="16.125" size="1.778" layer="27" rot="R180" display="off"/>
+<attribute name="MFG_PART_#" value="CRCW04021M00FKED" x="13.5" y="16.125" size="1.778" layer="27" rot="R180" display="off"/>
 <attribute name="TOLERANCE" value="±1%" x="13.5" y="16.125" size="1.778" layer="27" rot="R180" display="off"/>
 <attribute name="TEMP" value="±100ppm/°C" x="13.5" y="16.125" size="1.778" layer="27" rot="R180" display="off"/>
-<attribute name="USD" value="0.78/10" x="13.5" y="16.125" size="1.778" layer="27" rot="R180" display="off"/>
-<attribute name="DIGIKEY_PART_#" value="541-90.9KLCT-ND" x="13.5" y="16.125" size="1.778" layer="27" rot="R180" display="off"/>
+<attribute name="USD" value="2.11/50" x="13.5" y="16.125" size="1.778" layer="27" rot="R180" display="off"/>
+<attribute name="DIGIKEY_PART_#" value="541-1.00MLCT-ND" x="13.5" y="16.125" size="1.778" layer="27" rot="R180" display="off"/>
 </element>
-<element name="RAUXBOT" library="dubec" package="0402" value="RES2.94K_16" x="13.5" y="15" rot="R180">
-<attribute name="DIGIKEY_PART_#" value="541-2.94KLCT-ND" x="13.5" y="15" size="1.778" layer="27" rot="R180" display="off"/>
+<element name="RAUXBOT" library="dubec" package="0402" value="RES162K_16" x="13.5" y="15" rot="R180">
+<attribute name="DIGIKEY_PART_#" value="541-162KLCT-ND" x="13.5" y="15" size="1.778" layer="27" rot="R180" display="off"/>
 <attribute name="MANUFACTURER" value="Vishay Dale" x="13.5" y="15" size="1.778" layer="27" rot="R180" display="off"/>
-<attribute name="MFG_PART_#" value="CRCW04022K94FKED" x="13.5" y="15" size="1.778" layer="27" rot="R180" display="off"/>
+<attribute name="MFG_PART_#" value="CRCW0402162KFKED" x="13.5" y="15" size="1.778" layer="27" rot="R180" display="off"/>
 <attribute name="TOLERANCE" value="±1%" x="13.5" y="15" size="1.778" layer="27" rot="R180" display="off"/>
 <attribute name="TEMP" value="±100ppm/°C" x="13.5" y="15" size="1.778" layer="27" rot="R180" display="off"/>
